Commit message: add rgb camera and vlp16 lidar

File: scout/scout_description/urdf/scout_v2.xacro (robot description, xacro)
@@ -2,4 +2,9 @@
 <robot name="scout_v2"
     xmlns:xacro="http://ros.org/wiki/xacro">
+    <xacro:arg name="gpu" default="false"/>
+    <xacro:property name="gpu" value="$(arg gpu)" />
+    <xacro:arg name="organize_cloud" default="false"/>
+    <xacro:property name="organize_cloud" value="$(arg organize_cloud)" />
+    <xacro:arg name="camera_visual" default="false"/>
     <xacro:arg name="robot_namespace" default="/" />
     <xacro:arg name="urdf_extras" default="empty.urdf" />
@@ -84,3 +89,127 @@
     <!-- Gazebo definitions  -->
     <xacro:include filename="$(find scout_description)/urdf/scout_v2.gazebo" />
+    <!-- IMU e sensores -->
+    <!-- IMUUUU -->
+    <link name="imu_link"/>
+    <joint name="imu_joint" type="fixed">
+        <parent link="base_link"/>
+        <child link="imu_link"/>
+        <origin xyz="0.0 0 0.068" rpy="0 0 0"/>
+    </joint>
+    <!-- <gazebo reference="imu_link">
+        <sensor type="imu" name="imu">
+        <always_on>true</always_on>
+        <visualize>$(arg imu_visual)</visualize>
+        </sensor>
+        <material>Gazebo/Grey</material>
+    </gazebo> -->
+    <gazebo>
+        <plugin name="imu_plugin" filename="libgazebo_ros_imu.so">
+        <alwaysOn>true</alwaysOn>
+        <bodyName>imu_link</bodyName>
+        <frameName>imu_link</frameName>
+        <topicName>imu</topicName>
+        <serviceName>imu_service</serviceName>
+        <gaussianNoise>0.0</gaussianNoise>
+        <updateRate>0</updateRate>
+        <imu>
+            <noise>
+            <type>gaussian</type>
+            <rate>
+                <mean>0.0</mean>
+                <stddev>2e-4</stddev>
+                <bias_mean>0.0000075</bias_mean>
+                <bias_stddev>0.0000008</bias_stddev>
+            </rate>
+            <accel>
+                <mean>0.0</mean>
+                <stddev>1.7e-2</stddev>
+                <bias_mean>0.1</bias_mean>
+                <bias_stddev>0.001</bias_stddev>
+            </accel>
+            </noise>
+        </imu>
+        </plugin>
+    </gazebo>
+    <!-- VLP1666666 -->
+    <xacro:include filename="$(find velodyne_description)/urdf/VLP-16.urdf.xacro"/>
+    <xacro:VLP-16 parent="base_link" name="velodyne" topic="/velodyne_points" organize_cloud="${organize_cloud}" hz="10" samples="440" gpu="${gpu}">
+        <origin xyz="0 0 0.2" rpy="0 0 0" />
+    </xacro:VLP-16>
+    <!-- CAMERAAAAAAA -->
+    <link name="camera_link"/>
+    <joint name="camera_joint" type="fixed">
+        <parent link="base_link"/>
+        <child link="camera_link"/>
+        <origin xyz="0.0 0 0.4" rpy="0 0 0"/>
+    </joint>
+    <gazebo reference="camera_link">
+        <sensor type="camera" name="Pi Camera">
+            <always_on>true</always_on>
+            <visualize>$(arg camera_visual)</visualize>
+            <camera>
+                <horizontal_fov>1.085595</horizontal_fov>
+                <image>
+                    <width>640</width>
+                    <height>480</height>
+                    <format>R8G8B8</format>
+                </image>
+                <clip>
+                    <near>0.03</near>
+                    <far>100</far>
+                </clip>
+            </camera>
+            <plugin name="camera_controller" filename="libgazebo_ros_camera.so">
+                <alwaysOn>true</alwaysOn>
+                <updateRate>30.0</updateRate>
+                <cameraName>camera</cameraName>
+                <frameName>camera_link</frameName>
+                <imageTopicName>rgb/image_raw</imageTopicName>
+                <cameraInfoTopicName>rgb/camera_info</cameraInfoTopicName>
+                <hackBaseline>0.07</hackBaseline>
+                <distortionK1>0.0</distortionK1>
+                <distortionK2>0.0</distortionK2>
+                <distortionK3>0.0</distortionK3>
+                <distortionT1>0.0</distortionT1>
+                <distortionT2>0.0</distortionT2>
+            </plugin>
+        </sensor>
+    </gazebo>
+    <!-- STEREO CAMERAAAAAAA -->
+    <link name="stereo_camera_link">
+      <inertial>
+        <origin
+          xyz="1.8066E-07 -0.013922 -5.14669999914755E-09"
+          rpy="0 0 0" />
+        <mass
+          value="0.011423" />
+        <inertia
+          ixx="1.02528087587849E-06"
+          ixy="-2.77738904265723E-11"
+          ixz="-2.5418963856357E-12"
+          iyy="3.33817433207942E-05"
+          iyz="-7.17759958750659E-13"
+          izz="3.39466645935057E-05" />
+      </inertial>
+      <visual>
+        <origin xyz="0.0 0.0 0.0" rpy="1.57 0.0 1.57"/>
+        <geometry>
+          <mesh filename="package://scout_description/meshes/double-camera-mynt1.STL"/>
+        </geometry>
+      </visual>
+      <collision>
+        <origin
+          xyz="0 0 0"
+          rpy="1.57 0.0 1.57" />
+        <geometry>
+          <mesh
+            filename="package://scout_description/meshes/double-camera-mynt1.STL" />
+        </geometry>
+      </collision>
+    </link>
+    <joint name="stereo_camera_joint" type="fixed">
+        <parent link="base_link"/>
+        <child link="stereo_camera_link"/>
+        <origin xyz="0.0 0 0.3" rpy="0 0 0"/>
+    </joint>
 </robot>

Commit message: add stereo and depth plugin

File: scout/scout_description/urdf/scout_v2.xacro (robot description, xacro)
@@ -142,5 +142,5 @@
         <parent link="base_link"/>
         <child link="camera_link"/>
-        <origin xyz="0.0 0 0.4" rpy="0 0 0"/>
+        <origin xyz="0.3 0 0.4" rpy="0 0 0"/>
     </joint>
     <gazebo reference="camera_link">
@@ -211,5 +211,142 @@
         <parent link="base_link"/>
         <child link="stereo_camera_link"/>
-        <origin xyz="0.0 0 0.3" rpy="0 0 0"/>
-    </joint>
+        <origin xyz="0.3 0 0.3" rpy="0 0 0"/>
+    </joint>
+    <link name="left_stereo_camera_link" />
+    <joint name="left_stereo_camera_joint" type="fixed">
+      <parent link="stereo_camera_link" />
+      <child link="left_stereo_camera_link" />
+      <origin xyz="0.04 0.06 0" rpy="0 0 0"/>
+    </joint>
+    <link name="right_stereo_camera_link" />
+    <joint name="right_stereo_camera_joint" type="fixed">
+      <parent link="stereo_camera_link" />
+      <child link="right_stereo_camera_link" />
+      <origin xyz="0.04 -0.06 0" rpy="0 0 0"/>
+    </joint>
+    <link name="depth_stereo_camera_link" />
+    <joint name="depth_stereo_camera_joint" type="fixed">
+      <parent link="stereo_camera_link" />
+      <child link="depth_stereo_camera_link" />
+      <origin xyz="0.04 0 0" rpy="0 0 0"/>
+    </joint>
+    <!-- Camera stereo image plugin -->
+    <gazebo reference="left_stereo_camera_link">
+      <sensor type="multicamera" name="stereo_camera">
+        <update_rate>30.0</update_rate>
+        <camera name="left">
+          <horizontal_fov>2.1293</horizontal_fov>
+          <image>
+            <width>752</width>
+            <height>480</height>
+            <format>L8</format>
+          </image>
+          <clip>
+            <near>0.8</near>
+            <far>35</far>
+          </clip>
+          <noise>
+            <type>gaussian</type>
+            <mean>0.0</mean>
+            <stddev>0.007</stddev>
+          </noise>
+        </camera>
+        <camera name="right">
+          <pose frame="right_stereo_camera_link">0 0 0 0 0 0</pose>
+          <!-- <pose>0 -0.06 0 0 0 0</pose> -->
+          <horizontal_fov>2.1293</horizontal_fov>
+          <image>
+            <width>752</width>
+            <height>480</height>
+            <format>L8</format>
+          </image>
+          <clip>
+            <near>0.8</near>
+            <far>35</far>
+          </clip>
+          <noise>
+            <type>gaussian</type>
+            <mean>0.0</mean>
+            <stddev>0.007</stddev>
+          </noise>
+        </camera>
+        <plugin name="stereo_camera_controller" filename="libgazebo_ros_multicamera.so">
+          <alwaysOn>true</alwaysOn>
+          <updateRate>0.0</updateRate>
+          <cameraName>/stereo_camera</cameraName>
+          <imageTopicName>image_raw</imageTopicName>
+          <cameraInfoTopicName>stereo_camera_info</cameraInfoTopicName>
+          <frameName>left_stereo_camera_link</frameName>
+          <rightFrameName>right_stereo_camera_link</rightFrameName>
+          <!-- <frameName>/left_camera_optical_frame</frameName> -->
+          <!-- <rightFrameName>/right_camera_optical_frame</rightFrameName> -->
+          <hackBaseline>0.07</hackBaseline>
+          <distortionK1>0.0</distortionK1>
+          <distortionK2>0.0</distortionK2>
+          <distortionK3>0.0</distortionK3>
+          <distortionT1>0.0</distortionT1>
+          <distortionT2>0.0</distortionT2>
+        </plugin>
+      </sensor>
+    </gazebo>
+    <!-- Depth camera image plugin -->
+    <gazebo reference="depth_stereo_camera_link">
+      <sensor name="depth_camera" type="depth">
+        <update_rate>20</update_rate>
+        <camera>
+          <horizontal_fov>1.3962634</horizontal_fov>
+          <image>
+            <width>800</width>
+            <height>800</height>
+            <format>R8G8B8</format>
+          </image>
+          <clip>
+            <near>0.05</near>
+            <far>3</far>
+          </clip>
+        </camera>
+        <plugin name="depth_stereo_camera_controller" filename="libgazebo_ros_openni_kinect.so">
+          <baseline>0.2</baseline>
+          <alwaysOn>true</alwaysOn>
+          <updateRate>1.0</updateRate>
+          <cameraName>depth_camera_ir</cameraName>
+          <depthImageTopicName>depth/image_raw</depthImageTopicName>
+          <depthImageInfoTopicName>depth/camera_info</depthImageInfoTopicName>
+          <pointCloudTopicName>depth/points</pointCloudTopicName>
+          <frameName>depth_stereo_camera_link</frameName>
+          <pointCloudCutoff>0.5</pointCloudCutoff>
+          <pointCloudCutoffMax>3.0</pointCloudCutoffMax>
+          <distortionK1>0.00000001</distortionK1>
+          <distortionK2>0.00000001</distortionK2>
+          <distortionK3>0.00000001</distortionK3>
+          <distortionT1>0.00000001</distortionT1>
+          <distortionT2>0.00000001</distortionT2>
+          <CxPrime>0</CxPrime>
+          <Cx>0</Cx>
+          <Cy>0</Cy>
+          <focalLength>0</focalLength>
+          <hackBaseline>0</hackBaseline>
+        </plugin>
+      </sensor>
+    </gazebo>
+    <!-- GPSSSSS -->
+    <link name="gps_link" />
+    <joint name="gps_joint" type="fixed">
+        <parent link="base_link" />
+        <child link="gps_link" />
+        <origin xyz="0 0 0" rpy="0 0 0"/>
+    </joint>
+    <!-- <gazebo>
+        <plugin name="novatel_gps_sim" filename="libhector_gazebo_ros_gps.so">
+        <alwaysOn>1</alwaysOn>
+        <updateRate>10.0</updateRate>
+        <bodyName>base_link</bodyName>
+        <topicName>fix</topicName>
+        <velocityTopicName>fix_velocity</velocityTopicName>
+        <drift>5.0 5.0 5.0</drift>
+        <gaussianNoise>0.1 0.1 0.1</gaussianNoise>
+        <velocityDrift>0 0 0</velocityDrift>
+        <velocityGaussianNoise>0.1 0.1 0.1</velocityGaussianNoise>
+        </plugin>
+    </gazebo> -->
 </robot>

Commit message: fix depth camera

File: scout/scout_description/urdf/scout_v2.xacro (robot description, xacro)
@@ -225,10 +225,4 @@
       <origin xyz="0.04 -0.06 0" rpy="0 0 0"/>
     </joint>
-    <link name="depth_stereo_camera_link" />
-    <joint name="depth_stereo_camera_joint" type="fixed">
-      <parent link="stereo_camera_link" />
-      <child link="depth_stereo_camera_link" />
-      <origin xyz="0.04 0 0" rpy="0 0 0"/>
-    </joint>
     <!-- Camera stereo image plugin -->
     <gazebo reference="left_stereo_camera_link">
@@ -290,5 +284,19 @@
       </sensor>
     </gazebo>
-    <!-- Depth camera image plugin -->
+    <!-- depth camera link e joint  -->
+    <link name="depth_stereo_camera_link"/>
+    <joint name="depth_stereo_camera_joint" type="fixed">
+      <parent link="stereo_camera_link" />
+      <child link="depth_stereo_camera_link" />
+      <origin xyz="0.04 0 0" rpy="0 0 0"/>
+    </joint>
+    <!-- depth camera optical frame -->
+    <link name="depth_stereo_camera_optical_link"/>
+    <joint name="depth_stereo_camera_optical_joint" type="fixed">
+      <parent link="depth_stereo_camera_link" />
+      <child link="depth_stereo_camera_optical_link" />
+      <origin xyz="0 0 0" rpy="1.57 3.14 1.57"/>
+    </joint>
+    <!-- Depth camera image plugin 1 -->
     <gazebo reference="depth_stereo_camera_link">
       <sensor name="depth_camera" type="depth">
@@ -297,6 +305,8 @@
           <horizontal_fov>1.3962634</horizontal_fov>
           <image>
-            <width>800</width>
-            <height>800</height>
+            <!-- <width>800</width>
+            <height>800</height> -->
+            <width>640</width>
+            <height>480</height>
             <format>R8G8B8</format>
           </image>
@@ -314,5 +324,5 @@
           <depthImageInfoTopicName>depth/camera_info</depthImageInfoTopicName>
           <pointCloudTopicName>depth/points</pointCloudTopicName>
-          <frameName>depth_stereo_camera_link</frameName>
+          <frameName>depth_stereo_camera_optical_link</frameName>
           <pointCloudCutoff>0.5</pointCloudCutoff>
           <pointCloudCutoffMax>3.0</pointCloudCutoffMax>
@@ -337,16 +347,16 @@
         <origin xyz="0 0 0" rpy="0 0 0"/>
     </joint>
-    <!-- <gazebo>
-        <plugin name="novatel_gps_sim" filename="libhector_gazebo_ros_gps.so">
+    <gazebo>
+      <plugin name="novatel_gps_sim" filename="libhector_gazebo_ros_gps.so">
         <alwaysOn>1</alwaysOn>
         <updateRate>10.0</updateRate>
         <bodyName>base_link</bodyName>
-        <topicName>fix</topicName>
-        <velocityTopicName>fix_velocity</velocityTopicName>
+        <topicName>gps</topicName>
+        <velocityTopicName>gps_velocity</velocityTopicName>
         <drift>5.0 5.0 5.0</drift>
         <gaussianNoise>0.1 0.1 0.1</gaussianNoise>
         <velocityDrift>0 0 0</velocityDrift>
         <velocityGaussianNoise>0.1 0.1 0.1</velocityGaussianNoise>
-        </plugin>
-    </gazebo> -->
+      </plugin>
+    </gazebo>
 </robot>

Commit message: fix xacro files

File: scout/scout_description/urdf/scout_v2.xacro (robot description, xacro)
@@ -89,6 +89,11 @@
     <!-- Gazebo definitions  -->
     <xacro:include filename="$(find scout_description)/urdf/scout_v2.gazebo" />
-    <!-- IMU e sensores -->
-    <!-- IMUUUU -->
+    <!-- SENSORS AND INCLUDES ================================================ -->
+    <!-- SUBOT VLP16 INCLUDE -->
+    <xacro:include filename="$(find velodyne_description)/urdf/VLP-16.urdf.xacro"/>
+    <xacro:VLP-16 parent="base_link" name="velodyne" topic="/velodyne_points" organize_cloud="${organize_cloud}" hz="10" samples="440" gpu="${gpu}">
+        <origin xyz="0 0 0.2" rpy="0 0 0" />
+    </xacro:VLP-16>
+    <!-- SUBOT IMU frame-->
     <link name="imu_link"/>
     <joint name="imu_joint" type="fixed">
@@ -104,4 +109,5 @@
         <material>Gazebo/Grey</material>
     </gazebo> -->
+    <!-- SUBOT IMU PLUGIN -->
     <gazebo>
         <plugin name="imu_plugin" filename="libgazebo_ros_imu.so">
@@ -132,11 +138,6 @@
         </plugin>
     </gazebo>
-    <!-- VLP1666666 -->
-    <xacro:include filename="$(find velodyne_description)/urdf/VLP-16.urdf.xacro"/>
-    <xacro:VLP-16 parent="base_link" name="velodyne" topic="/velodyne_points" organize_cloud="${organize_cloud}" hz="10" samples="440" gpu="${gpu}">
-        <origin xyz="0 0 0.2" rpy="0 0 0" />
-    </xacro:VLP-16>
-    <!-- CAMERAAAAAAA -->
-    <link name="camera_link"/>
+    <!-- SUBOT RGB CAMERA (DISABLE) -->
+    <!-- <link name="camera_link"/>
     <joint name="camera_joint" type="fixed">
         <parent link="base_link"/>
@@ -175,6 +176,6 @@
             </plugin>
         </sensor>
-    </gazebo>
-    <!-- STEREO CAMERAAAAAAA -->
+    </gazebo>    -->
+    <!-- SUBOT STEREO CAMERA -->
     <link name="stereo_camera_link">
       <inertial>
@@ -225,5 +226,5 @@
       <origin xyz="0.04 -0.06 0" rpy="0 0 0"/>
     </joint>
-    <!-- Camera stereo image plugin -->
+    <!-- SUBOT STEREO CAMERA image plugin -->
     <gazebo reference="left_stereo_camera_link">
       <sensor type="multicamera" name="stereo_camera">
@@ -284,5 +285,5 @@
       </sensor>
     </gazebo>
-    <!-- depth camera link e joint  -->
+    <!-- SUBOT DEPTH CAMERA link and joint  -->
     <link name="depth_stereo_camera_link"/>
     <joint name="depth_stereo_camera_joint" type="fixed">
@@ -291,5 +292,5 @@
       <origin xyz="0.04 0 0" rpy="0 0 0"/>
     </joint>
-    <!-- depth camera optical frame -->
+    <!-- SUBOT DEPTH CAMERA optical frame -->
     <link name="depth_stereo_camera_optical_link"/>
     <joint name="depth_stereo_camera_optical_joint" type="fixed">
@@ -298,5 +299,5 @@
       <origin xyz="0 0 0" rpy="1.57 3.14 1.57"/>
     </joint>
-    <!-- Depth camera image plugin 1 -->
+    <!-- SUBOT DEPTH CAMERA image plugin -->
     <gazebo reference="depth_stereo_camera_link">
       <sensor name="depth_camera" type="depth">
@@ -340,5 +341,5 @@
       </sensor>
     </gazebo>
-    <!-- GPSSSSS -->
+    <!-- SUBOT GPS -->
     <link name="gps_link" />
     <joint name="gps_joint" type="fixed">
@@ -360,3 +361,16 @@
       </plugin>
     </gazebo>
+    <!-- SUBOT ODOMETRY -->
+    <gazebo>
+      <plugin name="p3d_base_controller" filename="libgazebo_ros_p3d.so">
+        <alwaysOn>true</alwaysOn>
+        <updateRate>50.0</updateRate>
+        <bodyName>base_link</bodyName>
+        <topicName>odom</topicName>
+        <gaussianNoise>0.01</gaussianNoise>
+        <frameName>world</frameName>
+        <xyzOffsets>0 0 0</xyzOffsets>
+        <rpyOffsets>0 0 0</rpyOffsets>
+      </plugin>
+    </gazebo>
 </robot>

Commit message: organize xacro file

File: scout/scout_description/urdf/scout_v2.xacro (robot description, xacro)
@@ -90,10 +90,17 @@
     <xacro:include filename="$(find scout_description)/urdf/scout_v2.gazebo" />
     <!-- SENSORS AND INCLUDES ================================================ -->
-    <!-- SUBOT VLP16 INCLUDE -->
+    <!-- SUBOT WORLD -->
+    <!-- <link name="world" />
+    <joint name="world_to_base_link=" type="planar">
+        <origin xyz="0 0 0.1" rpy="0 0 0" />
+        <parent link="world"/>
+        <child link="base_link"/>
+    </joint> -->
+    <!-- SUBOT VLP16 include -->
     <xacro:include filename="$(find velodyne_description)/urdf/VLP-16.urdf.xacro"/>
     <xacro:VLP-16 parent="base_link" name="velodyne" topic="/velodyne_points" organize_cloud="${organize_cloud}" hz="10" samples="440" gpu="${gpu}">
         <origin xyz="0 0 0.2" rpy="0 0 0" />
     </xacro:VLP-16>
-    <!-- SUBOT IMU frame-->
+    <!-- SUBOT IMU frame and joint -->
     <link name="imu_link"/>
     <joint name="imu_joint" type="fixed">
@@ -109,5 +116,5 @@
         <material>Gazebo/Grey</material>
     </gazebo> -->
-    <!-- SUBOT IMU PLUGIN -->
+    <!-- SUBOT IMU plugin -->
     <gazebo>
         <plugin name="imu_plugin" filename="libgazebo_ros_imu.so">
@@ -177,5 +184,5 @@
         </sensor>
     </gazebo>    -->
-    <!-- SUBOT STEREO CAMERA -->
+    <!-- SUBOT STEREO CAMERA  frames and joints -->
     <link name="stereo_camera_link">
       <inertial>
@@ -286,19 +293,19 @@
     </gazebo>
     <!-- SUBOT DEPTH CAMERA link and joint  -->
-    <link name="depth_stereo_camera_link"/>
-    <joint name="depth_stereo_camera_joint" type="fixed">
+    <link name="depth_camera_link"/>
+    <joint name="depth_camera_joint" type="fixed">
       <parent link="stereo_camera_link" />
-      <child link="depth_stereo_camera_link" />
+      <child link="depth_camera_link" />
       <origin xyz="0.04 0 0" rpy="0 0 0"/>
     </joint>
     <!-- SUBOT DEPTH CAMERA optical frame -->
-    <link name="depth_stereo_camera_optical_link"/>
-    <joint name="depth_stereo_camera_optical_joint" type="fixed">
-      <parent link="depth_stereo_camera_link" />
-      <child link="depth_stereo_camera_optical_link" />
+    <link name="depth_camera_optical_link"/>
+    <joint name="depth_camera_optical_joint" type="fixed">
+      <parent link="depth_camera_link" />
+      <child link="depth_camera_optical_link" />
       <origin xyz="0 0 0" rpy="1.57 3.14 1.57"/>
     </joint>
     <!-- SUBOT DEPTH CAMERA image plugin -->
-    <gazebo reference="depth_stereo_camera_link">
+    <gazebo reference="depth_camera_link">
       <sensor name="depth_camera" type="depth">
         <update_rate>20</update_rate>
@@ -317,13 +324,13 @@
           </clip>
         </camera>
-        <plugin name="depth_stereo_camera_controller" filename="libgazebo_ros_openni_kinect.so">
+        <plugin name="depth_camera_controller" filename="libgazebo_ros_openni_kinect.so">
           <baseline>0.2</baseline>
           <alwaysOn>true</alwaysOn>
           <updateRate>1.0</updateRate>
-          <cameraName>depth_camera_ir</cameraName>
+          <cameraName>depth_camera</cameraName>
           <depthImageTopicName>depth/image_raw</depthImageTopicName>
           <depthImageInfoTopicName>depth/camera_info</depthImageInfoTopicName>
           <pointCloudTopicName>depth/points</pointCloudTopicName>
-          <frameName>depth_stereo_camera_optical_link</frameName>
+          <frameName>depth_camera_optical_link</frameName>
           <pointCloudCutoff>0.5</pointCloudCutoff>
           <pointCloudCutoffMax>3.0</pointCloudCutoffMax>

Commit message: add rtab launch file

File: scout/scout_description/urdf/scout_v2.xacro (robot description, xacro)
@@ -201,5 +201,5 @@
       </inertial>
       <visual>
-        <origin xyz="0.0 0.0 0.0" rpy="1.57 0.0 1.57"/>
+        <origin xyz="0.0 0.0 0.0" rpy="${M_PI/2} 0.0 ${M_PI/2}"/>
         <geometry>
           <mesh filename="package://scout_description/meshes/double-camera-mynt1.STL"/>
@@ -209,5 +209,5 @@
         <origin
           xyz="0 0 0"
-          rpy="1.57 0.0 1.57" />
+          rpy="${M_PI/2} 0.0 ${M_PI/2}" />
         <geometry>
           <mesh
@@ -304,5 +304,5 @@
       <parent link="depth_camera_link" />
       <child link="depth_camera_optical_link" />
-      <origin xyz="0 0 0" rpy="1.57 3.14 1.57"/>
+      <origin xyz="0 0 0" rpy="${M_PI/2} ${M_PI} ${M_PI/2}"/>
     </joint>
     <!-- SUBOT DEPTH CAMERA image plugin -->
