Commit message: finish add and fix sensors

File: scout/scout_description/urdf/scout_v2.xacro (robot description, xacro)
@@ -90,31 +90,24 @@
     <xacro:include filename="$(find scout_description)/urdf/scout_v2.gazebo" />
     <!-- SENSORS AND INCLUDES ================================================ -->
-    <!-- SUBOT WORLD -->
+    <!-- WORLD -->
     <!-- <link name="world" />
-    <joint name="world_to_base_link=" type="planar">
-        <origin xyz="0 0 0.1" rpy="0 0 0" />
+    <joint name="world_to_base_link=" type="fixed">
+        <origin xyz="0 0 0.3" rpy="0 0 0" />
         <parent link="world"/>
         <child link="base_link"/>
     </joint> -->
-    <!-- SUBOT VLP16 include -->
+    <!-- VLP16 include -->
     <xacro:include filename="$(find velodyne_description)/urdf/VLP-16.urdf.xacro"/>
     <xacro:VLP-16 parent="base_link" name="velodyne" topic="/velodyne_points" organize_cloud="${organize_cloud}" hz="10" samples="440" gpu="${gpu}">
         <origin xyz="0 0 0.2" rpy="0 0 0" />
     </xacro:VLP-16>
-    <!-- SUBOT IMU frame and joint -->
+    <!-- IMU frame and joint -->
     <link name="imu_link"/>
     <joint name="imu_joint" type="fixed">
         <parent link="base_link"/>
         <child link="imu_link"/>
-        <origin xyz="0.0 0 0.068" rpy="0 0 0"/>
-    </joint>
-    <!-- <gazebo reference="imu_link">
-        <sensor type="imu" name="imu">
-        <always_on>true</always_on>
-        <visualize>$(arg imu_visual)</visualize>
-        </sensor>
-        <material>Gazebo/Grey</material>
-    </gazebo> -->
-    <!-- SUBOT IMU plugin -->
+        <origin xyz="0 0 0" rpy="0 0 0"/>
+    </joint>
+    <!-- IMU plugin -->
     <gazebo>
         <plugin name="imu_plugin" filename="libgazebo_ros_imu.so">
@@ -145,5 +138,5 @@
         </plugin>
     </gazebo>
-    <!-- SUBOT RGB CAMERA (DISABLE) -->
+    <!-- RGB CAMERA (DISABLE) -->
     <!-- <link name="camera_link"/>
     <joint name="camera_joint" type="fixed">
@@ -184,5 +177,5 @@
         </sensor>
     </gazebo>    -->
-    <!-- SUBOT STEREO CAMERA  frames and joints -->
+    <!-- STEREO CAMERA  frames and joints -->
     <link name="stereo_camera_link">
       <inertial>
@@ -233,5 +226,5 @@
       <origin xyz="0.04 -0.06 0" rpy="0 0 0"/>
     </joint>
-    <!-- SUBOT STEREO CAMERA image plugin -->
+    <!-- STEREO CAMERA image plugin -->
     <gazebo reference="left_stereo_camera_link">
       <sensor type="multicamera" name="stereo_camera">
@@ -292,5 +285,5 @@
       </sensor>
     </gazebo>
-    <!-- SUBOT DEPTH CAMERA link and joint  -->
+    <!-- DEPTH CAMERA link and joint  -->
     <link name="depth_camera_link"/>
     <joint name="depth_camera_joint" type="fixed">
@@ -299,5 +292,5 @@
       <origin xyz="0.04 0 0" rpy="0 0 0"/>
     </joint>
-    <!-- SUBOT DEPTH CAMERA optical frame -->
+    <!-- DEPTH CAMERA optical frame -->
     <link name="depth_camera_optical_link"/>
     <joint name="depth_camera_optical_joint" type="fixed">
@@ -306,5 +299,5 @@
       <origin xyz="0 0 0" rpy="${M_PI/2} ${M_PI} ${M_PI/2}"/>
     </joint>
-    <!-- SUBOT DEPTH CAMERA image plugin -->
+    <!-- DEPTH CAMERA image plugin -->
     <gazebo reference="depth_camera_link">
       <sensor name="depth_camera" type="depth">
@@ -348,5 +341,5 @@
       </sensor>
     </gazebo>
-    <!-- SUBOT GPS -->
+    <!-- GPS -->
     <link name="gps_link" />
     <joint name="gps_joint" type="fixed">
@@ -368,5 +361,5 @@
       </plugin>
     </gazebo>
-    <!-- SUBOT ODOMETRY -->
+    <!-- ODOMETRY -->
     <gazebo>
       <plugin name="p3d_base_controller" filename="libgazebo_ros_p3d.so">
@@ -376,5 +369,5 @@
         <topicName>odom</topicName>
         <gaussianNoise>0.01</gaussianNoise>
-        <frameName>world</frameName>
+        <frameName>map</frameName>
         <xyzOffsets>0 0 0</xyzOffsets>
         <rpyOffsets>0 0 0</rpyOffsets>

Commit message: Update Hunter and scout for ignition

File: scout/scout_description/urdf/scout_v2.xacro (robot description, xacro)
@@ -17,4 +17,11 @@
     <xacro:property name="wheel_length" value="1.1653e-01" />
     <xacro:property name="wheel_radius" value="1.6459e-01" />
+    <link name="base_footprint">
+    </link>
+    <joint name="base_footprint_to_base_link" type="fixed">
+        <origin xyz="0 0 0.23" rpy="0 0 0" />
+        <parent link="base_footprint" />
+        <child link="base_link" />
+    </joint>
     <!-- Base link -->
     <link name="base_link">
@@ -58,4 +65,72 @@
         <child link="inertial_link" />
     </joint>
+     <!-- ================== IMU ================== -->
+  <link name="imu_link">
+    <inertial>
+      <mass value="0.05"/>
+      <origin rpy="0 0 0" xyz="0 0 0"/>
+      <inertia ixx="1e-6" ixy="0" ixz="0" iyy="1e-6" iyz="0" izz="1e-6"/>
+    </inertial>
+    <visual>
+      <origin rpy="0 0 0" xyz="0 0 0"/>
+      <geometry>
+        <box size="0.02 0.02 0.02"/>
+      </geometry>
+      <material name="imu_green">
+        <color rgba="0.2 0.8 0.2 1.0"/>
+      </material>
+    </visual>
+  </link>
+  <joint name="imu_joint" type="fixed">
+    <parent link="base_link"/>
+    <!-- posicione a IMU no chassis -->
+    <child link="imu_link"/>
+    <origin rpy="0 0 0" xyz="0 0 0.1"/>
+  </joint>
+  <!-- ================== LiDAR 3D ================== -->
+  <link name="lidar_3d_link">
+    <inertial>
+      <mass value="0.3"/>
+      <origin rpy="0 0 0" xyz="0 0 0"/>
+      <inertia ixx="1e-4" ixy="0" ixz="0" iyy="1e-4" iyz="0" izz="1e-4"/>
+    </inertial>
+    <visual>
+      <origin rpy="0 0 0" xyz="0 0 0"/>
+      <geometry>
+        <cylinder length="0.06" radius="0.05"/>
+      </geometry>
+      <material name="lidar_black">
+        <color rgba="0.1 0.1 0.1 1.0"/>
+      </material>
+    </visual>
+  </link>
+  <joint name="lidar_3d_joint" type="fixed">
+    <parent link="base_link"/>
+    <!-- posicione a IMU no chassis -->
+    <child link="lidar_3d_link"/>
+    <origin rpy="0 0 0" xyz="0 0 0.25"/>
+  </joint>
+  <!-- ================== LiDAR 2D ================== -->
+  <link name="lidar_2d_link">
+    <inertial>
+      <mass value="0.3"/>
+      <origin rpy="0 0 0" xyz="0 0 0"/>
+      <inertia ixx="1e-4" ixy="0" ixz="0" iyy="1e-4" iyz="0" izz="1e-4"/>
+    </inertial>
+    <visual>
+      <origin rpy="0 0 0" xyz="0 0 0"/>
+      <geometry>
+        <cylinder length="0.06" radius="0.05"/>
+      </geometry>
+      <material name="lidar_black">
+        <color rgba="0.1 0.1 0.1 1.0"/>
+      </material>
+    </visual>
+  </link>
+  <joint name="lidar_2d_joint" type="fixed">
+    <parent link="base_link"/>
+    <child link="lidar_2d_link"/>
+    <origin rpy="0 0 0" xyz="0.55 0 -0.10"/>
+  </joint>
     <!-- For testing, hang the robot up in the air -->
     <!-- <link name="world" />

Commit message: Update skidsteer controller

File: scout/scout_description/urdf/scout_v2.xacro (robot description, xacro)
@@ -18,4 +18,9 @@
     <xacro:property name="wheel_radius" value="1.6459e-01" />
     <link name="base_footprint">
+      <inertial>
+        <origin xyz="0 0 0" rpy="0 0 0"/>
+        <mass value="0.001"/>
+        <inertia ixx="1e-6" ixy="0" ixz="0" iyy="1e-6" iyz="0" izz="1e-6"/>
+      </inertial>
     </link>
     <joint name="base_footprint_to_base_link" type="fixed">
@@ -133,4 +138,18 @@
     <origin rpy="0 0 0" xyz="0.55 0 -0.10"/>
   </joint>
+  <link name="camera_rgbd_link"/>
+  <joint name="camera_rgbd_joint" type="fixed">
+    <parent link="base_link"/>
+    <child link="camera_rgbd_link"/>
+    <!-- ajuste a pose na frente do robô -->
+    <origin xyz="0.35 0.0 0.25" rpy="0 0 0"/>
+  </joint>
+  <link name="camera_rgbd_optical_frame"/>
+  <joint name="camera_rgbd_optical_joint" type="fixed">
+    <parent link="camera_rgbd_link"/>
+    <child link="camera_rgbd_optical_frame"/>
+    <!-- rotação para virar optical frame (REP-103) -->
+    <origin xyz="0 0 0" rpy="-1.57079632679 0 -1.57079632679"/>
+  </joint>
     <!-- For testing, hang the robot up in the air -->
     <!-- <link name="world" />
